File: pcb/rev.A/sizif512.sch (KiCad schematic (older format))
At the start: 206 parts, among them J1 DS1020-05, J10 Mini-DIN-9, J11 PJ-313, J12 PJ-313, J13 Conn_02x28_Row_Letter_First, J14 Conn_01x10, J15 MEM2055-00-190-01-A, J2 DS-210, J3 DS1020-08, J4 Conn_01x04, J5 Conn_02x05, J6 Conn_02x05_Odd_Even, J7 DB9-M, J8 Conn_02x05_Odd_Even, J9 Conn_02x17_Odd_Even, Q1 IRF9540, Q2 BC547B, Q3 BC547B, Q4 BC547C, Q5 BC547B, Q6 BC547B, Q7 BC547B, Q8 BC547B, SW1 SW_SPST, SW2 SW_Push, SW3 SW_Push, U1 74HCU04, U10 EPM3256ATC144-10, U11 AS6C4008-55PCN, U12 MB8877A, U13 AY-3-8310, U2 MAX314CSE/DG413DY, U3 74HC04, U4 74HC4050, U5 LM311, U6 L7805, U7 Z84C0010PEC, U8 AMS1117-3.3, U9 SST39SF040, Y1 14.318MHz, Y2 32MHz

Commit message: update rev.A pcb
Parts:
- J4: value Conn_01x04 -> WF-4
- LS1: value Speaker -> WF-2
- R22: value 100k -> 470k
- R91: value 2.2k -> 1.5k
- R92: value 8.2k -> 5.6k
- SW2: value SW_Push -> WF-2
- SW3: value SW_Push -> WF-2; Desc CONFIG -> MAGIC
- U13: value AY-3-8310 -> AY-3-8910
- U5: value LM311 -> LM311N
- U6: value L7805 -> K78L05-1000R3
Connections:
- no-connect marks 39 -> 38
Other:
- note added: "CLOCK"
- note added: "PORTS"
- note removed: "CLOCK GENERATOR"
- moved on the sheet: C26, C27, C28, C29, C30, C31, C32, C33, C34, C35, C36, C37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
