File: pcb/rev.B/sizif512.kicad_pcb (KiCad board)
At the start: 2 copper layers, 213 x 65.1 mm, 214 parts, among them J1 Conn_01x05, J10 DB9-M, J11 Conn_02x05_Odd_Even, J12 Mini-DIN-9, J13 RCJ-014, J14 PJ-313, J15 PJ-313, J16 Conn_02x28_Row_Letter_First, J17 Conn_01x10, J18 MEM2055-00-190-01-A, J2 Conn_01x08, J3 DS-210, J4 WF-4, J5 JTAG, J6 Conn_01x02, J7 Conn_02x05_Top_Bottom, J8 Conn_01x02, J9 Conn_02x17_Odd_Even, Q1 BC547B, Q2 BC547C, Q3 BC547C, Q4 BC547C, Q5 BC547C, SW1 Conn_01x02, SW2 WF-2, SW3 WF-2, U1 74HCU04, U10 1818VG93, U11 EPM3256ATC144, U12 AS6C4008-55PCN, U13 74HCT4053D, U14 AY-3-8310, U15 AD724, U2 74HCT05, U3 74HCU04, U4 Z84C0008PEC, U5 L4940V5 / K7805-2000R3L, U6 AM1S-0512SZ, U7 AMS1117-3.3, U8 LM2596T-ADJ, U9 29C040, Y1 17.734475 MHz, Y2 8 MHz

Commit message: add rev.B (abandoned) and rev.C (wip) pcbs
Routing:
- net GND: track 970.8 -> 902.2 mm
Changed lines of the file:
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@@
     (thickness 1.6)
     (drawings 45)
-    (tracks 4079)
+    (tracks 4076)
     (zones 0)
     (modules 214)
@@
   (segment (start 48.641 71.25312) (end 51.19688 71.25312) (width 1) (layer B.Cu) (net 1))
   (segment (start 109.7872 95.9878) (end 111.8128 95.9878) (width 1) (layer F.Cu) (net 1))
-  (segment (start 128.228 127.052) (end 90.128 127.052) (width 1) (layer F.Cu) (net 1))
   (segment (start 136.0004 127.052) (end 137.1484 128.2) (width 0.2) (layer B.Cu) (net 1))
   (segment (start 137.1484 128.2) (end 137.45 128.2) (width 0.2) (layer B.Cu) (net 1))
@@
   (segment (start 119.1 95.98) (end 119.1078 95.9878) (width 1) (layer F.Cu) (net 1))
   (segment (start 118.2378 95.98) (end 119.1 95.98) (width 1) (layer F.Cu) (net 1))
-  (segment (start 130.768 127.052) (end 128.228 127.052) (width 1) (layer F.Cu) (net 1))
   (via (at 129.49 108.67) (size 0.8) (drill 0.4) (layers F.Cu B.Cu) (net 1))
   (segment (start 119.1078 95.9878) (end 119.973991 96.853991) (width 1) (layer F.Cu) (net 1))
@@
   (via (at 245.684 119.032) (size 0.8) (drill 0.4) (layers F.Cu B.Cu) (net 1))
   (via (at 245.684 117.212) (size 0.8) (drill 0.4) (layers F.Cu B.Cu) (net 1))
-  (segment (start 90.128 127.052) (end 118.068 127.052) (width 1) (layer B.Cu) (net 1))
   (segment (start 49.61 113.22) (end 54.805 113.22) (width 1) (layer F.Cu) (net 1))
   (segment (start 49.51 128.72) (end 52.005 128.72) (width 1) (layer F.Cu) (net 1))
