File: pcb_wifi/rev.A/sizif512-wifi.kicad_pcb (KiCad board)
At the start: 2 copper layers, 24 x 34 mm, 13 parts, among them J1 Conn_01x10, U1 AP1117-33, U2 ESP-12E

Commit message: add rev.B (abandoned) and rev.C (wip) pcbs
Parts:
- U1: value AP1117-33 -> AMS1117-3.3
Changed lines of the file:
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@@
       (effects (font (size 1 1) (thickness 0.15)))
     )
-    (fp_text value AP1117-33 (at -2.9 0 180) (layer F.Fab)
+    (fp_text value AMS1117-3.3 (at -2.9 0 180) (layer F.Fab)
       (effects (font (size 1 1) (thickness 0.15)))
     )
