File: pcb_wifi/rev.A/sizif512-wifi.sch (KiCad schematic (older format))
At the start: 13 parts, among them J1 Conn_01x10, U1 AP1117-33, U2 ESP-12E

Commit message: add rev.B (abandoned) and rev.C (wip) pcbs
Parts:
- U1: value AP1117-33 -> AMS1117-3.3; symbol Regulator_Linear:AP1117-33 -> Regulator_Linear:AMS1117-3.3
Changed lines of the file:
@@
 $EndComp
 $Comp
-L Regulator_Linear:AP1117-33 U1
+L Regulator_Linear:AMS1117-3.3 U1
 U 1 1 5EA457DB
 P 6175 2875
 F 0 "U1" H 6175 3117 50  0000 C CNN
-F 1 "AP1117-33" H 6175 3026 50  0000 C CNN
+F 1 "AMS1117-3.3" H 6175 3026 50  0000 C CNN
 F 2 "Package_TO_SOT_SMD:SOT-223-3_TabPin2" H 6175 3075 50  0001 C CNN
 F 3 "http://www.diodes.com/datasheets/AP1117.pdf" H 6275 2625 50  0001 C CNN
