File: pcb/rev.C/sizif512.kicad_pcb (KiCad board)
At the start: 2 copper layers, 213 x 65 mm, 186 parts, among them J1 DS-210, J10 RCJ-014, J11 PinHeader, J12 PJ-313, J13 PinHeader, J14 PinHeader, J15 PJ-313, J16 MEM2055-00-190-01-A, J17 PinHeader, J2 Conn_02x28_Row_Letter_First, J3 PinHeader, J4 DS1020-08, J5 DS1020-05, J6 PinHeader, J7 DB9-M, J8 PinHeader, J9 Mini-DIN-9, Q1 BC547C, Q2 BC547C, Q3 BC547C, Q4 BC547C, SW1 Jumper, SW2 Button THT, SW3 Button THT, U1 LM2596T-ADJ, U10 SN74CB3T3245PW, U11 AD724, U12 AS6C4008-55PCN, U13 74HCT4053D, U14 AY-3-8910, U15 LM311N, U2 AMS1117-3.3, U3 SN74CB3T3245PW, U4 Z84C0010PEC, U5 SN74CB3T3245PW, U6 EPM1270T144, U7 SN74CB3T3245PW, U8 SST39SF040, U9 74HCU04, Y1 28 MHz, Y2 4.433 MHz

Commit message: pcb rev.C: minor layout changes
Parts:
- C18: value 100n -> 10n
- C41, C42: value 1n -> 4.7n
Routing:
- net /SND_DAC_L: track 26.7 -> 23.8 mm
- net Net-(D2-Pad2): track 39.3 -> 37.7 mm
- net /~RFSH: track 122.3 -> 121.5 mm
- net /A6: track 99.5 -> 100.1 mm
- net /~NMI: track 109.6 -> 109.1 mm
