File: pcb/rev.C1/sizif512.kicad_pcb (KiCad board)
At the start: 2 copper layers, 213 x 65 mm, 186 parts, among them J1 DS-210, J10 RCJ-014, J11 PinHeader, J12 PJ-313, J13 PinHeader, J14 PinHeader, J15 PJ-313, J16 MEM2055-00-190-01-A, J17 PinHeader, J2 Conn_02x28_Row_Letter_First, J3 PinHeader, J4 DS1020-08, J5 DS1020-05, J6 PinHeader, J7 DB9-M, J8 PinHeader, J9 Mini-DIN-9, Q1 BC547C, Q2 BC547C, Q3 BC547C, Q4 BC547C, SW1 Jumper, SW2 Button THT, SW3 Button THT, U1 LM2596T-ADJ, U10 SN74CB3T3245PW, U11 AD724, U12 AS6C4008-55PCN, U13 74HCT4053D, U14 AY-3-8910, U15 LM311N, U2 AMS1117-3.3, U3 SN74CB3T3245PW, U4 Z84C0010PEC, U5 SN74CB3T3245PW, U6 EPM1270T144, U7 SN74CB3T3245PW, U8 SST39SF040, U9 74HCU04, Y1 28 MHz, Y2 4.433 MHz

Commit message: pcb rev.C1: minor values change
Video circuit tuning:
R10, R17, R22, R26, R27, R27: 1.5k
R12, R20, R25: 3k
C43: 30p (wider range is better)
Q1, Q2, Q3, Q4: BC549B (low noise, less amplification)

Exclude 2.2k value from BOM:
R6, R7: 2k

Also add some assembly drawing.
Parts:
- C43: value 10p -> 30p
- Q1, Q2, Q3, Q4: value BC547C -> BC549B
- R10, R17, R22: value 3.6k -> 1.5k
- R12, R20, R25: value 9.1k -> 3k
- R26, R27, R28: value 4.7k -> 1.5k
- R6, R7: value 2.2k -> 2k
Other:
- board text added: "Install horizontally"
- board text added: "Install one of J6 or J7"
- board text added: "Install one of J9 or J10"
- board text added: "Install one of SW2 or J14"
- board text added: "Install one of SW3 or J17"

Commit message: pcb rev.C1: update Y1 capacitors values for better reliability
Parts:
- C35, C36: value 6p -> 22p
Changed lines of the file:
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@@
       (effects (font (size 0.8 1) (thickness 0.15)))
     )
-    (fp_text value 6p (at 1.7484 -0.1176 180) (layer F.Fab)
+    (fp_text value 22p (at 1.7484 -0.1176 180) (layer F.Fab)
       (effects (font (size 0.6 0.6) (thickness 0.1)))
     )
@@
       (effects (font (size 0.8 1) (thickness 0.15)))
     )
-    (fp_text value 6p (at 1.7384 -0.0376 180) (layer F.Fab)
+    (fp_text value 22p (at 1.7384 -0.0376 180) (layer F.Fab)
       (effects (font (size 0.6 0.6) (thickness 0.1)))
     )
